Commit message: chore: Restructure the data directory
- Move all reachy data to data/reachy
- This is because we will add other robots in the future
- Change the mesh path of reachy.urdf

File: data/reachy/reachy.urdf (robot description, URDF)
Before this commit: robot reachy, 31 links, 30 joints
Links:
- link bottom_neck_arm: geometry collision cylinder length=0.0 radius=0.0; visual mesh filename=data/reachy/reachy_meshes/orbita_arm.obj
- link head: geometry collision cylinder length=0.15 radius=0.06; visual mesh filename=data/reachy/reachy_meshes/head.obj
- link l_antenna_link: geometry collision cylinder length=0.0 radius=0.0; visual mesh filename=data/reachy/reachy_meshes/antenna.obj
- link l_forearm: geometry collision cylinder length=0.09 radius=0.04; visual mesh filename=data/reachy/reachy_meshes/forearm.obj
- link l_gripper_finger: geometry collision box size=0.1 0.012 0.035; visual mesh filename=data/reachy/reachy_meshes/l_gripper_finger.obj
- link l_gripper_thumb: geometry collision box size=0.1 0.012 0.035; visual mesh filename=data/reachy/reachy_meshes/l_gripper_thumb.obj
- link l_shoulder: geometry collision cylinder length=0.09 radius=0.035; visual mesh filename=data/reachy/reachy_meshes/shoulder.obj
- link l_shoulder_x: geometry collision cylinder length=0.04 radius=0.035; visual mesh filename=data/reachy/reachy_meshes/shoulder_x.obj
- link l_upper_arm: geometry collision cylinder length=0.25 radius=0.04; visual mesh filename=data/reachy/reachy_meshes/upper_arm.obj
- link l_wrist: geometry collision cylinder length=0.14 radius=0.035; visual mesh filename=data/reachy/reachy_meshes/wrist.obj
- link l_wrist2hand: geometry collision cylinder length=0.06 radius=0.03; visual mesh filename=data/reachy/reachy_meshes/wrist2hand.obj
- link middle_neck_arm: geometry collision cylinder length=0.0 radius=0.0; visual mesh filename=data/reachy/reachy_meshes/orbita_arm.obj
- link r_antenna_link: geometry collision cylinder length=0.0 radius=0.0; visual mesh filename=data/reachy/reachy_meshes/antenna.obj
- link r_forearm: geometry collision cylinder length=0.09 radius=0.04; visual mesh filename=data/reachy/reachy_meshes/forearm.obj
- link r_gripper_finger: geometry collision box size=0.1 0.012 0.035; visual mesh filename=data/reachy/reachy_meshes/r_gripper_finger.obj
- link r_gripper_thumb: geometry collision box size=0.1 0.012 0.035; visual mesh filename=data/reachy/reachy_meshes/r_gripper_thumb.obj
- link r_shoulder: geometry collision cylinder length=0.09 radius=0.035; visual mesh filename=data/reachy/reachy_meshes/shoulder.obj
- link r_shoulder_x: geometry collision cylinder length=0.04 radius=0.035; visual mesh filename=data/reachy/reachy_meshes/shoulder_x.obj
- link r_upper_arm: geometry collision cylinder length=0.25 radius=0.04; visual mesh filename=data/reachy/reachy_meshes/upper_arm.obj
- link r_wrist: geometry collision cylinder length=0.14 radius=0.035; visual mesh filename=data/reachy/reachy_meshes/wrist.obj
- link r_wrist2hand: geometry collision cylinder length=0.06 radius=0.03; visual mesh filename=data/reachy/reachy_meshes/wrist2hand.obj
- link top_neck_arm: geometry collision cylinder length=0.0 radius=0.0; visual mesh filename=data/reachy/reachy_meshes/orbita_arm.obj
- link torso: geometry collision box size=0.11 0.2 0.32; visual mesh filename=data/reachy/reachy_meshes/torso.obj
