Commit message: chore: add data for robots
- 문제가 있는 상태이지만 정리를 위해 일단 커밋

File: data/coman/model.urdf (robot description, URDF)
Before this commit: robot coman, 66 links, 65 joints
Links:
- link LFootmot: geometry collision mesh filename=./meshes/simple/Leg4.STL scale=0.03937 -0.03937 0.03937; visual mesh filename=./meshes/Leg4.STL scale=0.03937 0.03937 0.03937
- link LHipMot: geometry collision mesh filename=./meshes/simple/Leg0.STL scale=0.03937 -0.03937 0.03937; visual mesh filename=./meshes/Leg0.STL scale=0.03937 0.03937 0.03937
- link LLowLeg: geometry collision mesh filename=./meshes/simple/Leg3.STL scale=0.03937 -0.03937 0.03937; visual mesh filename=./meshes/Leg3.STL scale=0.03937 0.03937 0.03937
- link LShr: geometry collision mesh filename=./meshes/simple/Arm1.STL scale=0.03937 -0.03937 0.03937; visual mesh filename=./meshes/Arm1.STL scale=0.03937 0.03937 0.03937
- link LShy: geometry collision mesh filename=./meshes/simple/Arm2.STL scale=0.03937 -0.03937 0.03937; visual mesh filename=./meshes/Arm2.STL scale=0.03937 0.03937 0.03937
- link LSoftHand: geometry collision mesh filename=./meshes/simple/SoftHandOpen.STL scale=-1E-3 1E-3 1E-3; visual mesh filename=./meshes/SoftHandOpen.STL scale=-0.1 0.1 -0.1
- link LThighLowLeg: geometry collision mesh filename=./meshes/simple/Leg2.STL scale=0.03937 -0.03937 0.03937; visual mesh filename=./meshes/Leg2.STL scale=0.03937 0.03937 0.03937
- link LThighUpLeg: geometry collision mesh filename=./meshes/simple/Leg1.STL scale=0.03937 -0.03937 0.03937; visual mesh filename=./meshes/Leg1.STL scale=0.03937 0.03937 0.03937

File: data/reachy/reachy.urdf (robot description, URDF)
Before this commit: robot reachy, 31 links, 30 joints
Links:
- link bottom_neck_arm: geometry collision cylinder length=0.0 radius=0.0; visual mesh filename=./reachy_meshes/orbita_arm.obj
- link head: geometry collision cylinder length=0.15 radius=0.06; visual mesh filename=./reachy_meshes/head.obj
- link l_antenna_link: geometry collision cylinder length=0.0 radius=0.0; visual mesh filename=./reachy_meshes/antenna.obj
- link l_forearm: geometry collision cylinder length=0.09 radius=0.04; visual mesh filename=./reachy_meshes/forearm.obj
- link l_gripper_finger: geometry collision box size=0.1 0.012 0.035; visual mesh filename=./reachy_meshes/l_gripper_finger.obj
- link l_gripper_thumb: geometry collision box size=0.1 0.012 0.035; visual mesh filename=./reachy_meshes/l_gripper_thumb.obj
- link l_shoulder: geometry collision cylinder length=0.09 radius=0.035; visual mesh filename=./reachy_meshes/shoulder.obj
- link l_shoulder_x: geometry collision cylinder length=0.04 radius=0.035; visual mesh filename=./reachy_meshes/shoulder_x.obj
- link l_upper_arm: geometry collision cylinder length=0.25 radius=0.04; visual mesh filename=./reachy_meshes/upper_arm.obj
- link l_wrist: geometry collision cylinder length=0.14 radius=0.035; visual mesh filename=./reachy_meshes/wrist.obj
- link l_wrist2hand: geometry collision cylinder length=0.06 radius=0.03; visual mesh filename=./reachy_meshes/wrist2hand.obj
- link middle_neck_arm: geometry collision cylinder length=0.0 radius=0.0; visual mesh filename=./reachy_meshes/orbita_arm.obj
- link r_antenna_link: geometry collision cylinder length=0.0 radius=0.0; visual mesh filename=./reachy_meshes/antenna.obj
- link r_forearm: geometry collision cylinder length=0.09 radius=0.04; visual mesh filename=./reachy_meshes/forearm.obj
- link r_gripper_finger: geometry collision box size=0.1 0.012 0.035; visual mesh filename=./reachy_meshes/r_gripper_finger.obj
- link r_gripper_thumb: geometry collision box size=0.1 0.012 0.035; visual mesh filename=./reachy_meshes/r_gripper_thumb.obj
- link r_shoulder: geometry collision cylinder length=0.09 radius=0.035; visual mesh filename=./reachy_meshes/shoulder.obj
- link r_shoulder_x: geometry collision cylinder length=0.04 radius=0.035; visual mesh filename=./reachy_meshes/shoulder_x.obj
- link r_upper_arm: geometry collision cylinder length=0.25 radius=0.04; visual mesh filename=./reachy_meshes/upper_arm.obj
- link r_wrist: geometry collision cylinder length=0.14 radius=0.035; visual mesh filename=./reachy_meshes/wrist.obj
- link r_wrist2hand: geometry collision cylinder length=0.06 radius=0.03; visual mesh filename=./reachy_meshes/wrist2hand.obj
- link top_neck_arm: geometry collision cylinder length=0.0 radius=0.0; visual mesh filename=./reachy_meshes/orbita_arm.obj
- link torso: geometry collision box size=0.11 0.2 0.32; visual mesh filename=./reachy_meshes/torso.obj

File: data/reachy/reachy2.urdf (robot description, URDF)
Before this commit: robot reachy, 31 links, 30 joints
Links:
- link head: geometry collision cylinder length=0.15 radius=0.06; visual mesh filename=./reachy_meshes/head.obj
- link l_antenna_link: geometry collision cylinder length=0.0 radius=0.0; visual mesh filename=./reachy_meshes/antenna.obj
- link l_shoulder: geometry collision cylinder length=0.09 radius=0.035; visual mesh filename=./reachy_meshes/shoulder.obj
- link l_shoulder_x: geometry collision cylinder length=0.04 radius=0.035; visual mesh filename=./reachy_meshes/shoulder_x.obj
- link l_wrist: geometry collision cylinder length=0.14 radius=0.035; visual mesh filename=./reachy_meshes/wrist.obj
- link l_wrist2hand: geometry collision cylinder length=0.06 radius=0.03; visual mesh filename=./reachy_meshes/wrist2hand.obj
- link r_antenna_link: geometry collision cylinder length=0.0 radius=0.0; visual mesh filename=./reachy_meshes/antenna.obj
- link r_forearm: geometry collision cylinder length=0.09 radius=0.04; visual mesh filename=./reachy_meshes/forearm.obj
- link r_gripper_finger: geometry collision box size=0.1 0.012 0.035; visual mesh filename=./reachy_meshes/r_gripper_finger.obj
- link r_gripper_thumb: geometry collision box size=0.1 0.012 0.035; visual mesh filename=./reachy_meshes/r_gripper_thumb.obj
- link r_shoulder: geometry collision cylinder length=0.09 radius=0.035; visual mesh filename=./reachy_meshes/shoulder.obj
- link r_shoulder_x: geometry collision cylinder length=0.04 radius=0.035; visual mesh filename=./reachy_meshes/shoulder_x.obj
- link r_upper_arm: geometry collision cylinder length=0.25 radius=0.04; visual mesh filename=./reachy_meshes/upper_arm.obj
- link r_wrist: geometry collision cylinder length=0.14 radius=0.035; visual mesh filename=./reachy_meshes/wrist.obj
- link r_wrist2hand: geometry collision cylinder length=0.06 radius=0.03; visual mesh filename=./reachy_meshes/wrist2hand.obj
- link torso: geometry collision box size=0.11 0.2 0.32; visual mesh filename=./reachy_meshes/torso.obj
