Commit message: feat: add NAO's urdf & mesh file

File: data/nao/nao.urdf (robot description, URDF)
Before this commit: robot NaoH25V32, 77 links, 76 joints
Links:
- removed link CameraBottom_frame
- removed link CameraBottom_optical_frame
- removed link CameraTop_frame
- removed link CameraTop_optical_frame
- removed link ChestButton_frame
- removed link HeadTouchFront_frame
- removed link HeadTouchMiddle_frame
- removed link HeadTouchRear_frame
- removed link ImuTorsoAccelerometer_frame
- removed link ImuTorsoGyrometer_frame
- removed link LFootBumperLeft_frame
- removed link LFootBumperRight_frame
- removed link LFsrFL_frame
- removed link LFsrFR_frame
- removed link LFsrRL_frame
- removed link LFsrRR_frame
- removed link LInfraRed_frame
- removed link LSonar_frame
- removed link MicroFrontCenter_frame
- removed link MicroRearCenter_frame
- removed link MicroSurroundLeft_frame
- removed link MicroSurroundRight_frame
- removed link RFootBumperLeft_frame
- removed link RFootBumperRight_frame
- removed link RFsrFL_frame
- removed link RFsrFR_frame
- removed link RFsrRL_frame
- removed link RFsrRR_frame
- removed link RInfraRed_frame
- removed link RSonar_frame
- removed link gaze
- removed link l_sole
- removed link r_sole
- added link world
- link Head: mass 0.47672 -> 0.60533; geometry collision mesh filename=./visual/HeadPitch.stl scale=0.1 0.1 0.1; visual mesh filename=./visual/HeadPitch.stl scale=0.1 0.1 0.1
- link LAnklePitch: mass 0.13892 -> 0.13416; geometry collision mesh filename=./visual/LAnklePitch.stl scale=0.1 0.1 0.1; visual mesh filename=./visual/LAnklePitch.stl scale=0.1 0.1 0.1
- link LBicep: mass 0.12166 -> 0.15777; geometry collision mesh filename=./visual/LShoulderRoll.stl scale=0.1 0.1 0.1; visual mesh filename=./visual/LShoulderRoll.stl scale=0.1 0.1 0.1
- link LElbow: mass 0.05959 -> 0.06483
- link LFinger11_link: geometry collision mesh filename=./visual/LFinger11.stl scale=0.1 0.1 0.1; visual mesh filename=./visual/LFinger11.stl scale=0.1 0.1 0.1
- link LFinger12_link: geometry collision mesh filename=./visual/LFinger12.stl scale=0.1 0.1 0.1; visual mesh filename=./visual/LFinger12.stl scale=0.1 0.1 0.1
- link LFinger13_link: geometry collision mesh filename=./visual/LFinger13.stl scale=0.1 0.1 0.1; visual mesh filename=./visual/LFinger13.stl scale=0.1 0.1 0.1
- link LFinger21_link: geometry collision mesh filename=./visual/LFinger21.stl scale=0.1 0.1 0.1; visual mesh filename=./visual/LFinger21.stl scale=0.1 0.1 0.1
- link LFinger22_link: geometry collision mesh filename=./visual/LFinger22.stl scale=0.1 0.1 0.1; visual mesh filename=./visual/LFinger22.stl scale=0.1 0.1 0.1
- link LFinger23_link: geometry collision mesh filename=./visual/LFinger23.stl scale=0.1 0.1 0.1; visual mesh filename=./visual/LFinger23.stl scale=0.1 0.1 0.1
- link LForeArm: mass 0.0377 -> 0.07761; geometry collision mesh filename=./visual/LElbowRoll.stl scale=0.1 0.1 0.1; visual mesh filename=./visual/LElbowRoll.stl scale=0.1 0.1 0.1
- link LHip: mass 0.1353 -> 0.13053; geometry collision mesh filename=./visual/LHipRoll.stl scale=0.1 0.1 0.1; visual mesh filename=./visual/LHipRoll.stl scale=0.1 0.1 0.1
- link LPelvis: mass 0.07244 -> 0.06981; geometry collision mesh filename=./visual/LHipYawPitch.stl scale=0.1 0.1 0.1; visual mesh filename=./visual/LHipYawPitch.stl scale=0.1 0.1 0.1
- link LShoulder: mass 0.06984 -> 0.07504; geometry collision mesh filename=./visual/LShoulderPitch.stl scale=0.1 0.1 0.1; visual mesh filename=./visual/LShoulderPitch.stl scale=0.1 0.1 0.1
- link LThigh: mass 0.39798 -> 0.38968; geometry collision mesh filename=./visual/LHipPitch.stl scale=0.1 0.1 0.1; visual mesh filename=./visual/LHipPitch.stl scale=0.1 0.1 0.1
- link LThumb1_link: geometry collision mesh filename=./visual/LThumb1.stl scale=0.1 0.1 0.1; visual mesh filename=./visual/LThumb1.stl scale=0.1 0.1 0.1
- link LThumb2_link: geometry collision mesh filename=./visual/LThumb2.stl scale=0.1 0.1 0.1; visual mesh filename=./visual/LThumb2.stl scale=0.1 0.1 0.1
- link LTibia: mass 0.29714 -> 0.29142; geometry collision mesh filename=./visual/LKneePitch.stl scale=0.1 0.1 0.1; visual mesh filename=./visual/LKneePitch.stl scale=0.1 0.1 0.1
- link Neck: mass 0.05959 -> 0.06442; geometry collision mesh filename=./visual/HeadYaw.stl scale=0.1 0.1 0.1; visual mesh filename=./visual/HeadYaw.stl scale=0.1 0.1 0.1
- link RAnklePitch: mass 0.13892 -> 0.13416; geometry collision mesh filename=./visual/RAnklePitch.stl scale=0.1 0.1 0.1; visual mesh filename=./visual/RAnklePitch.stl scale=0.1 0.1 0.1
- link RBicep: mass 0.12166 -> 0.15777; geometry collision mesh filename=./visual/RShoulderRoll.stl scale=0.1 0.1 0.1; visual mesh filename=./visual/RShoulderRoll.stl scale=0.1 0.1 0.1
- link RElbow: mass 0.05959 -> 0.06483
- link RFinger11_link: geometry collision mesh filename=./visual/RFinger11.stl scale=0.1 0.1 0.1; visual mesh filename=./visual/RFinger11.stl scale=0.1 0.1 0.1
- link RFinger12_link: geometry collision mesh filename=./visual/RFinger12.stl scale=0.1 0.1 0.1; visual mesh filename=./visual/RFinger12.stl scale=0.1 0.1 0.1
- link RFinger13_link: geometry collision mesh filename=./visual/RFinger13.stl scale=0.1 0.1 0.1; visual mesh filename=./visual/RFinger13.stl scale=0.1 0.1 0.1
- link RFinger21_link: geometry collision mesh filename=./visual/RFinger21.stl scale=0.1 0.1 0.1; visual mesh filename=./visual/RFinger21.stl scale=0.1 0.1 0.1
- link RFinger22_link: geometry collision mesh filename=./visual/RFinger22.stl scale=0.1 0.1 0.1; visual mesh filename=./visual/RFinger22.stl scale=0.1 0.1 0.1
- link RFinger23_link: geometry collision mesh filename=./visual/RFinger23.stl scale=0.1 0.1 0.1; visual mesh filename=./visual/RFinger23.stl scale=0.1 0.1 0.1
- link RForeArm: mass 0.0377 -> 0.07761; geometry collision mesh filename=./visual/RElbowRoll.stl scale=0.1 0.1 0.1; visual mesh filename=./visual/RElbowRoll.stl scale=0.1 0.1 0.1
- link RHip: mass 0.1353 -> 0.13053; geometry collision mesh filename=./visual/RHipRoll.stl scale=0.1 0.1 0.1; visual mesh filename=./visual/RHipRoll.stl scale=0.1 0.1 0.1
- link RPelvis: mass 0.07244 -> 0.06981; geometry collision mesh filename=./visual/RHipYawPitch.stl scale=0.1 0.1 0.1; visual mesh filename=./visual/RHipYawPitch.stl scale=0.1 0.1 0.1
- link RShoulder: mass 0.06984 -> 0.07504; geometry collision mesh filename=./visual/RShoulderPitch.stl scale=0.1 0.1 0.1; visual mesh filename=./visual/RShoulderPitch.stl scale=0.1 0.1 0.1
- link RThigh: mass 0.39798 -> 0.38968; geometry collision mesh filename=./visual/RHipPitch.stl scale=0.1 0.1 0.1; visual mesh filename=./visual/RHipPitch.stl scale=0.1 0.1 0.1
- link RThumb1_link: geometry collision mesh filename=./visual/RThumb1.stl scale=0.1 0.1 0.1; visual mesh filename=./visual/RThumb1.stl scale=0.1 0.1 0.1
- link RThumb2_link: geometry collision mesh filename=./visual/RThumb2.stl scale=0.1 0.1 0.1; visual mesh filename=./visual/RThumb2.stl scale=0.1 0.1 0.1
- link RTibia: mass 0.29714 -> 0.29142; geometry collision mesh filename=./visual/RKneePitch.stl scale=0.1 0.1 0.1; visual mesh filename=./visual/RKneePitch.stl scale=0.1 0.1 0.1
- link l_ankle: mass 0.16304 -> 0.16184; geometry collision mesh filename=./visual/LAnkleRoll.stl scale=0.1 0.1 0.1; visual mesh filename=./visual/LAnkleRoll.stl scale=0.1 0.1 0.1
- link l_wrist: mass 0.14314 -> 0.18533; geometry collision mesh filename=./visual/LWristYaw.stl scale=0.1 0.1 0.1; visual mesh filename=./visual/LWristYaw.stl scale=0.1 0.1 0.1
- link r_ankle: mass 0.16304 -> 0.16184; geometry collision mesh filename=./visual/RAnkleRoll.stl scale=0.1 0.1 0.1; visual mesh filename=./visual/RAnkleRoll.stl scale=0.1 0.1 0.1
- link r_wrist: mass 0.14314 -> 0.18533; geometry collision mesh filename=./visual/RWristYaw.stl scale=0.1 0.1 0.1; visual mesh filename=./visual/RWristYaw.stl scale=0.1 0.1 0.1
- link torso: mass 1.02628 -> 1.04956; geometry collision mesh filename=./visual/Torso.stl scale=0.1 0.1 0.1; visual mesh filename=./visual/Torso.stl scale=0.1 0.1 0.1
Joints:
- removed joint Accelerometer_sensor_fixedjoint
- removed joint CameraBottom_optical_frame_fixedjoint
- removed joint CameraBottom_sensor_fixedjoint
- removed joint CameraTop_optical_frame_fixedjoint
- removed joint CameraTop_sensor_fixedjoint
- removed joint ChestBoard/Button_sensor_fixedjoint
- removed joint Gyrometer_sensor_fixedjoint
- removed joint Head/Touch/Front_sensor_fixedjoint
- removed joint Head/Touch/Middle_sensor_fixedjoint
- removed joint Head/Touch/Rear_sensor_fixedjoint
- removed joint InfraredL_sensor_fixedjoint
- removed joint InfraredR_sensor_fixedjoint
- removed joint LFoot/Bumper/Left_sensor_fixedjoint
- removed joint LFoot/Bumper/Right_sensor_fixedjoint
- removed joint LFoot/FSR/FrontLeft_sensor_fixedjoint
- removed joint LFoot/FSR/FrontRight_sensor_fixedjoint
- removed joint LFoot/FSR/RearLeft_sensor_fixedjoint
- removed joint LFoot/FSR/RearRight_sensor_fixedjoint
- removed joint LLeg_effector_fixedjoint
- removed joint MicroFront_sensor_fixedjoint
- removed joint MicroLeft_sensor_fixedjoint
- removed joint MicroRear_sensor_fixedjoint
- removed joint MicroRight_sensor_fixedjoint
- removed joint RFoot/Bumper/Left_sensor_fixedjoint
- removed joint RFoot/Bumper/Right_sensor_fixedjoint
- removed joint RFoot/FSR/FrontLeft_sensor_fixedjoint
- removed joint RFoot/FSR/FrontRight_sensor_fixedjoint
- removed joint RFoot/FSR/RearLeft_sensor_fixedjoint
- removed joint RFoot/FSR/RearRight_sensor_fixedjoint
- removed joint RLeg_effector_fixedjoint
- removed joint Sonar/Left_sensor_fixedjoint
- removed joint Sonar/Right_sensor_fixedjoint
- removed joint gaze_joint
- added joint world_fixed: type fixed, parent world, child base_link, origin xyz=0 0 0 rpy=0 0 0
- joint LElbowRoll: limit lower=-1.56207 upper=-0.00872665 effort=1.532 velocity=7.19407 -> lower=-1.54462 upper=-0.0349066 effort=1.532 velocity=7.19407
- joint LElbowYaw: origin xyz=0.09 0 0 rpy=0 0 0 -> xyz=0.105 0.015 0 rpy=0 0 0
- joint LHand: limit lower=0 upper=1.0 effort=0.292 velocity=3.71 -> lower=0 upper=1.0 effort=0.292 velocity=8.33; origin xyz=0.058 0 -0.0159 rpy=0 0 0 -> xyz=0.05775 0 -0.01231 rpy=0 0 0; type revolute -> fixed
- joint LShoulderRoll: limit lower=0.00872665 upper=1.64934 effort=1.7835 velocity=7.19407 -> lower=-0.314159 upper=1.32645 effort=1.7835 velocity=7.19407
- joint LWristYaw: limit lower=-1.82387 upper=1.82387 effort=0.3891 velocity=5.03144 -> lower=-1.82387 upper=1.82387 effort=0.4075 velocity=24.6229; origin xyz=0.05055 0 0 rpy=0 0 0 -> xyz=0.05595 0 0 rpy=0 0 0
- joint RElbowRoll: limit lower=0.00872665 upper=1.56207 effort=1.532 velocity=7.19407 -> lower=0.0349066 upper=1.54462 effort=1.532 velocity=7.19407
- joint RElbowYaw: origin xyz=0.09 0 0 rpy=0 0 0 -> xyz=0.105 -0.015 0 rpy=0 0 0
- joint RHand: limit lower=0 upper=1.0 effort=0.292 velocity=3.71 -> lower=0 upper=1.0 effort=0.292 velocity=8.33; origin xyz=0.058 0 -0.0159 rpy=0 0 0 -> xyz=0.05775 0 -0.01213 rpy=0 0 0; type revolute -> fixed
- joint RShoulderRoll: limit lower=-1.64934 upper=-0.00872665 effort=1.783 velocity=7.19407 -> lower=-1.32645 upper=0.314159 effort=1.783 velocity=7.19407
- joint RWristYaw: limit lower=-1.82387 upper=1.82387 effort=0.3891 velocity=5.03144 -> lower=-1.82387 upper=1.82387 effort=0.4075 velocity=24.6229; origin xyz=0.05055 0 0 rpy=0 0 0 -> xyz=0.05595 0 0 rpy=0 0 0
- joint base_link_fixedjoint: origin xyz=0 0 0 rpy=0 0 0 -> xyz=0 0 0.33 rpy=0 0 0
